Commit message: Fix urdf

File: nkinematics-urdf/sample.urdf (robot description, URDF)
Before this commit: robot robo, 7 links, 6 joints
Joints:
- joint elbow_pitch: origin xyz=0.0, 0.0, -0.2 -> xyz=0.0 0.0 -0.2
- joint shoulder_roll: origin xyz=0.0, 0.1, 0.0 -> xyz=0.0 0.1 0.0
- joint wrist_pitch: origin xyz=0.0, 0.0, -0.2 -> xyz=0.0 0.0 -0.2
- joint wrist_yaw: origin xyz=0.0, 0.0, -0.2 -> xyz=0.0 0.0 -0.2

Commit message: Support for multiple LinkedFrames

File: nkinematics-urdf/sample.urdf (robot description, URDF)
Before this commit: robot robo, 7 links, 6 joints
Links:
- removed link elbow1
- removed link shoulder1
- removed link shoulder2
- removed link shoulder3
- removed link wrist1
- removed link wrist2
- added link l_elbow1; visual box size=0.1 0.1 0.2
- added link l_shoulder1; visual box size=0.1 0.1 0.1
- added link l_shoulder2; visual box size=0.1 0.1 0.1
- added link l_shoulder3; visual box size=0.1 0.1 0.2
- added link l_wrist1; visual box size=0.1 0.15 0.1
- added link l_wrist2; visual box size=0.05 0.08 0.15
- added link r_elbow1; visual box size=0.1 0.1 0.2
- added link r_shoulder1; visual box size=0.1 0.1 0.1
- added link r_shoulder2; visual box size=0.1 0.1 0.1
- added link r_shoulder3; visual box size=0.1 0.1 0.2
- added link r_wrist1; visual box size=0.1 0.15 0.1
- added link r_wrist2; visual box size=0.05 0.08 0.15
- link root: mass None -> 1; geometry collision cylinder length=0.5 radius=1; visual box size=0.2 0.2 0.4
Joints:
- removed joint elbow_pitch
- removed joint shoulder_pitch
- removed joint shoulder_roll
- removed joint shoulder_yaw
- removed joint wrist_pitch
- removed joint wrist_yaw
- added joint l_elbow_pitch: type revolute, parent l_shoulder3, child l_elbow1, origin xyz=0.0 0.0 -0.2, axis 0 1 0, limit lower=-2 upper=1.0 effort=0 velocity=1.0
- added joint l_shoulder_pitch: type revolute, parent l_shoulder1, child l_shoulder2, origin xyz=0.0 0.1 0.0, axis 0 1 0, limit lower=-1 upper=1.0 effort=0 velocity=1.0
- added joint l_shoulder_roll: type revolute, parent l_shoulder2, child l_shoulder3, origin xyz=0.0 0.1 0.0, axis 1 0 0, limit lower=-2 upper=1.0 effort=0 velocity=1.0
- added joint l_shoulder_yaw: type revolute, parent root, child l_shoulder1, origin xyz=0.0 0.2 0.2, axis 0 0 1, limit lower=-1 upper=1.0 effort=0 velocity=1.0
- added joint l_wrist_pitch: type revolute, parent l_wrist1, child l_wrist2, origin xyz=0.0 0.0 -0.2, axis 0 1 0, limit lower=-2 upper=1.0 effort=0 velocity=1.0
- added joint l_wrist_yaw: type revolute, parent l_elbow1, child l_wrist1, origin xyz=0.0 0.0 -0.2, axis 0 0 1, limit lower=-2 upper=1.0 effort=0 velocity=1.0
- added joint r_elbow_pitch: type revolute, parent r_shoulder3, child r_elbow1, origin xyz=0.0 0.0 -0.2, axis 0 1 0, limit lower=-2 upper=1.0 effort=0 velocity=1.0
- added joint r_shoulder_pitch: type revolute, parent r_shoulder1, child r_shoulder2, origin xyz=0.0 -0.1 0.0, axis 0 1 0, limit lower=-1 upper=1.0 effort=0 velocity=1.0
- added joint r_shoulder_roll: type revolute, parent r_shoulder2, child r_shoulder3, origin xyz=0.0 -0.1 0.0, axis 1 0 0, limit lower=-2 upper=1.0 effort=0 velocity=1.0
- added joint r_shoulder_yaw: type revolute, parent root, child r_shoulder1, origin xyz=0.0 -0.2 0.2, axis 0 0 1, limit lower=-1 upper=1.0 effort=0 velocity=1.0
- added joint r_wrist_pitch: type revolute, parent r_wrist1, child r_wrist2, origin xyz=0.0 0.0 -0.2, axis 0 1 0, limit lower=-2 upper=1.0 effort=0 velocity=1.0
- added joint r_wrist_yaw: type revolute, parent r_elbow1, child r_wrist1, origin xyz=0.0 0.0 -0.2, axis 0 0 1, limit lower=-2 upper=1.0 effort=0 velocity=1.0
